File: hardware/stepping-stone.kicad_sch (KiCad schematic)
At the start: 0 parts

Commit message: Begin TMC2209 sheet
Other:
- added sheet Stepper Driver 0 (tmc2209_driver.kicad_sch)
- note removed: "ESTOP?"
