File: hardware/sd_card.kicad_sch (KiCad schematic)
At the start: 19 parts, among them J4 Micro_SD_Card_Det_Hirose_DM3AT

Commit message: Minor Changes
Parts:
- D14: value ESD9B3.3ST5G -> ESD9B3
Changed lines of the file:
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@@
 			)
 		)
-		(property "Value" "ESD9B3.3ST5G"
+		(property "Value" "ESD9B3"
 			(at 115.57 124.46 90)
 			(show_name no)
