File: hardware/buck-converter.kicad_sch (KiCad schematic)
At the start: 13 parts

Commit message: Add QSPI Flash
Parts:
- gave numbers to parts that had none: 13
Changed lines of the file:
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@@
 		(in_pos_files yes)
 		(dnp no)
-		(property "Reference" "C?"
+		(property "Reference" "C6"
 			(at 113.03 93.9862 0)
 			(show_name no)
@@
 			(project "stepping-stone"
 				(path "/793a882e-3f7b-468b-a863-41a1f527e1bf/f256c00d-2170-4eef-a13f-c3325a813e7e"
-					(reference "C?")
+					(reference "C6")
 					(unit 1)
 				)
@@
 		(dnp no)
 		(fields_autoplaced yes)
-		(property "Reference" "R?"
+		(property "Reference" "R13"
 			(at 171.45 114.2999 0)
 			(show_name no)
@@
 			(project "stepping-stone"
 				(path "/793a882e-3f7b-468b-a863-41a1f527e1bf/f256c00d-2170-4eef-a13f-c3325a813e7e"
-					(reference "R?")
+					(reference "R13")
 					(unit 1)
 				)
@@
 		(dnp no)
 		(fields_autoplaced yes)
-		(property "Reference" "D?"
+		(property "Reference" "D7"
 			(at 186.69 115.8874 90)
 			(show_name no)
@@
 			(project "stepping-stone"
 				(path "/793a882e-3f7b-468b-a863-41a1f527e1bf/f256c00d-2170-4eef-a13f-c3325a813e7e"
-					(reference "D?")
+					(reference "D7")
 					(unit 1)
 				)
@@
 		(in_pos_files yes)
 		(dnp no)
-		(property "Reference" "C?"
+		(property "Reference" "C8"
 			(at 198.12 104.14 0)
 			(show_name no)
@@
 			(project "stepping-stone"
 				(path "/793a882e-3f7b-468b-a863-41a1f527e1bf/f256c00d-2170-4eef-a13f-c3325a813e7e"
-					(reference "C?")
+					(reference "C8")
 					(unit 1)
 				)
@@
 		(in_pos_files yes)
 		(dnp no)
-		(property "Reference" "D?"
+		(property "Reference" "D6"
 			(at 73.9775 90.17 0)
 			(show_name no)
@@
 			(project "stepping-stone"
 				(path "/793a882e-3f7b-468b-a863-41a1f527e1bf/f256c00d-2170-4eef-a13f-c3325a813e7e"
-					(reference "D?")
+					(reference "D6")
 					(unit 1)
 				)
@@
 		(dnp no)
 		(fields_autoplaced yes)
-		(property "Reference" "Q?"
+		(property "Reference" "Q2"
 			(at 134.62 82.55 0)
 			(show_name no)
@@
 			(project "stepping-stone"
 				(path "/793a882e-3f7b-468b-a863-41a1f527e1bf/f256c00d-2170-4eef-a13f-c3325a813e7e"
-					(reference "Q?")
+					(reference "Q2")
 					(unit 1)
 				)
@@
 		(in_pos_files yes)
 		(dnp no)
-		(property "Reference" "C?"
+		(property "Reference" "C5"
 			(at 100.965 93.9799 0)
 			(show_name no)
@@
 			(project "stepping-stone"
 				(path "/793a882e-3f7b-468b-a863-41a1f527e1bf/f256c00d-2170-4eef-a13f-c3325a813e7e"
-					(reference "C?")
+					(reference "C5")
 					(unit 1)
 				)
@@
 		(dnp no)
 		(fields_autoplaced yes)
-		(property "Reference" "R?"
+		(property "Reference" "R11"
 			(at 171.45 104.1399 0)
 			(show_name no)
@@
 			(project "stepping-stone"
 				(path "/793a882e-3f7b-468b-a863-41a1f527e1bf/f256c00d-2170-4eef-a13f-c3325a813e7e"
-					(reference "R?")
+					(reference "R11")
 					(unit 1)
 				)
@@
 		(in_pos_files yes)
 		(dnp no)
-		(property "Reference" "C?"
+		(property "Reference" "C9"
 			(at 215.9 104.14 0)
 			(show_name no)
@@
 			(project "stepping-stone"
 				(path "/793a882e-3f7b-468b-a863-41a1f527e1bf/f256c00d-2170-4eef-a13f-c3325a813e7e"
-					(reference "C?")
+					(reference "C9")
 					(unit 1)
 				)
@@
 		(dnp no)
 		(fields_autoplaced yes)
-		(property "Reference" "L?"
+		(property "Reference" "L1"
 			(at 160.02 95.25 90)
 			(show_name no)
@@
 			(project "stepping-stone"
 				(path "/793a882e-3f7b-468b-a863-41a1f527e1bf/f256c00d-2170-4eef-a13f-c3325a813e7e"
-					(reference "L?")
+					(reference "L1")
 					(unit 1)
 				)
@@
 		(dnp no)
 		(fields_autoplaced yes)
-		(property "Reference" "R?"
+		(property "Reference" "R12"
 			(at 185.42 104.1399 0)
 			(show_name no)
@@
 			(project "stepping-stone"
 				(path "/793a882e-3f7b-468b-a863-41a1f527e1bf/f256c00d-2170-4eef-a13f-c3325a813e7e"
-					(reference "R?")
+					(reference "R12")
 					(unit 1)
 				)
@@
 		(in_pos_files yes)
 		(dnp no)
-		(property "Reference" "C?"
+		(property "Reference" "C7"
 			(at 149.86 93.9862 0)
 			(show_name no)
@@
 			(project "stepping-stone"
 				(path "/793a882e-3f7b-468b-a863-41a1f527e1bf/f256c00d-2170-4eef-a13f-c3325a813e7e"
-					(reference "C?")
+					(reference "C7")
 					(unit 1)
 				)
@@
 		(in_pos_files yes)
 		(dnp no)
-		(property "Reference" "D?"
+		(property "Reference" "D5"
 			(at 73.9775 77.47 0)
 			(show_name no)
@@
 			(project "stepping-stone"
 				(path "/793a882e-3f7b-468b-a863-41a1f527e1bf/f256c00d-2170-4eef-a13f-c3325a813e7e"
-					(reference "D?")
+					(reference "D5")
 					(unit 1)
 				)

Commit message: Added Limit Switch Page
Other:
- note added: "1A MAX Output Current"
Changed lines of the file:
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@@
 		(company "Jacob Wigent")
+	)
+	(text "1A MAX Output Current"
+		(exclude_from_sim no)
+		(at 191.77 97.79 0)
+		(effects
+			(font
+				(size 1.27 1.27)
+			)
+		)
 	)
 	(junction

Commit message: Limit Switches and CAN Bus
Parts:
- Q2: value LMR51610YFDBVR -> LMR51625XDDCR; Part Number LMR51610YFDBVR -> LMR51625XDDCR; Vendor URL https://www.digikey.com/en/products/detail/texas-instruments/LMR51610YFDBVR/22286738 -> https://www.digikey.com/en/products/detail/texas-instruments/LMR51625XDDCR/25991371
Other:
- note added: "LMR51610YFDBVR = 1A MAX LMR51625XDDCR = 2.5A MAX"
- note removed: "1A MAX Output Current"
Changed lines of the file:
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@@
 		(company "Jacob Wigent")
 	)
-	(text "1A MAX Output Current"
+	(text "LMR51610YFDBVR = 1A MAX\nLMR51625XDDCR = 2.5A MAX"
 		(exclude_from_sim no)
-		(at 191.77 97.79 0)
+		(at 193.04 96.52 0)
 		(effects
 			(font
@@
 			)
 		)
-		(property "Value" "LMR51610YFDBVR"
+		(property "Value" "LMR51625XDDCR"
 			(at 134.62 85.09 0)
 			(show_name no)
@@
 			)
 		)
-		(property "Datasheet" "https://www.ti.com/lit/ds/symlink/lmr51610.pdf?ts=1708678595808&ref_url=https%253A%252F%252Fwww.ti.com%252Fproduct%252FLMR51610"
+		(property "Datasheet" "https://www.ti.com/lit/ds/symlink/lmr51625.pdf?ts=1742888310253&ref_url=https%253A%252F%252Fwww.ti.com%252Fsitesearch%252Fen-us%252Fdocs%252Funiversalsearch.tsp%253FlangPref%253Den-US%2526nr%253D3%2526searchTerm%253DLMR51625XDDCR"
 			(at 134.62 80.01 0)
 			(hide yes)
@@
 			)
 		)
-		(property "Description" "Buck Switching Regulator IC Positive Adjustable 0.8V 1 Output 0.6-1A SOT-23-6"
+		(property "Description" "Buck Switching Regulator IC Positive Adjustable 0.8V 1 Output 2.5A SOT-23-6 Thin, TSOT-23-6"
 			(at 134.62 80.01 0)
 			(hide yes)
@@
 			)
 		)
-		(property "Part Number" "LMR51610YFDBVR"
+		(property "Part Number" "LMR51625XDDCR"
 			(at 134.62 100.33 0)
 			(hide yes)
@@
 			)
 		)
-		(property "Vendor URL" "https://www.digikey.com/en/products/detail/texas-instruments/LMR51610YFDBVR/22286738"
+		(property "Vendor URL" "https://www.digikey.com/en/products/detail/texas-instruments/LMR51625XDDCR/25991371"
 			(at 134.62 100.33 0)
 			(hide yes)

Commit message: Fix Designators (Q -> U)
Parts:
- renumbered Q2 to U?
Changed lines of the file:
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@@
 		(dnp no)
 		(fields_autoplaced yes)
-		(property "Reference" "Q2"
+		(property "Reference" "U?"
 			(at 134.62 82.55 0)
 			(show_name no)
@@
 			(project "stepping-stone"
 				(path "/793a882e-3f7b-468b-a863-41a1f527e1bf/f256c00d-2170-4eef-a13f-c3325a813e7e"
-					(reference "Q2")
+					(reference "U?")
 					(unit 1)
 				)
