File: hardware/microcontroller.kicad_sch (KiCad schematic)
At the start: 19 parts, among them J2 STLink Header, SW1 BOOT, SW2 RESET, SW3 USER0, SW4 USER2, SW5 USER1, SW6 USER3, U1 STM32G474QBT6

Commit message: Finish aux i2c, uart, gpio
Changed lines of the file:
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@@
+		)
+	)
+	(hierarchical_label "AUX_SDA"
+		(shape bidirectional)
+		(at 350.52 110.49 0)
+		(effects
+			(font
+				(size 1.27 1.27)
+			)
+			(justify left)
 		)
 	)
@@
 		)
 	)
+	(hierarchical_label "AUX_SCL"
+		(shape bidirectional)
+		(at 350.52 113.03 0)
+		(effects
+			(font
+				(size 1.27 1.27)
+			)
+			(justify left)
+		)
+	)

Commit message: Aux IO Changes
Parts:
- added D? (x2): BLUE, Diode_SMD:D_0805_2012Metric, symbol Device:LED
- added D?: GREEN, Diode_SMD:D_0805_2012Metric, symbol Device:LED
- added D?: YELLOW, Diode_SMD:D_0805_2012Metric, symbol Device:LED
- added R? (x2): 220, Resistor_SMD:R_0603_1608Metric, symbol Device:R_US
- added R? (x2): 1k, Resistor_SMD:R_0603_1608Metric, symbol Device:R_US
Connections:
- net GND: now also D?.1 (K), D?.1 (K), D?.1 (K), D?.1 (K)
- net USER0 renamed USER_BTN_0
- net USER1 renamed USER_BTN_1
- net USER2 renamed USER_BTN_2
- net USER3 renamed USER_BTN_3
- new net: D?.2 (A), R?.2 (x4)
- new net USER_LED_0: R?.1
- new net USER_LED_1: R?.1
- new net USER_LED_2: R?.1
- new net USER_LED_3: R?.1
Other:
- note added: "User LEDs/Buttons"
- note removed: "Connector Search"
- note removed: "STLink v3 Minie connector"
- note removed: "User Buttons"
- note removed: "Would be hard to disconnect cable"
- moved on the sheet: C3, C4, D3, J2, R2, R3, R4, R5, R6, R7, R8, R9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
