File: hardware/qspi_flash.kicad_sch (KiCad schematic)
At the start: 3 parts

Commit message: Limit Switches and CAN Bus
Other:
- company: (none) -> Jacob Wigent
- title: (none) -> QSPI Flash
- moved on the sheet: C?, R?

Commit message: Add EEPROM
Parts:
- added C?: 0.1uF, Capacitor_SMD:C_0603_1608Metric_Pad1.08x0.95mm_HandSolder, symbol Device:C_Small
- added JP?: E1, Jumper:SolderJumper-3_P1.3mm_Bridged12_RoundedPad1.0x1.5mm, symbol Jumper:SolderJumper_3_Bridged12
- added JP?: ~{EC}, Jumper:SolderJumper-2_P1.3mm_Bridged_RoundedPad1.0x1.5mm, symbol Jumper:SolderJumper_2_Bridged
- added JP?: E0, Jumper:SolderJumper-3_P1.3mm_Bridged12_RoundedPad1.0x1.5mm, symbol Jumper:SolderJumper_3_Bridged12
- added JP?: E2, Jumper:SolderJumper-3_P1.3mm_Bridged12_RoundedPad1.0x1.5mm, symbol Jumper:SolderJumper_3_Bridged12
- added R? (x2): 2.2k, Resistor_SMD:R_0603_1608Metric, symbol Device:R_US
- added R?: 10k, Resistor_SMD:R_0603_1608Metric, symbol Device:R_US
- added U?: M24C02-FDW, Package_SO:TSSOP-8_4.4x3mm_P0.65mm, symbol Memory_EEPROM:M24C02-FDW
Connections:
- net +3.3V: now also C?.1, JP?.3 (B), JP?.3 (B), JP?.3 (B), R?.2, R?.2, U?.8 (VCC)
- net GND: now also C?.2, JP?.1 (A), JP?.1 (A), JP?.1 (A), R?.2, U?.4 (VSS)
- new net: JP?.2 (C), U?.2 (E1)
- new net: JP?.2 (B), R?.1, U?.7 (~{WC})
- new net: JP?.2 (C), U?.1 (E0)
- new net: JP?.2 (C), U?.3 (E2)
- new net SCL: R?.1, U?.6 (SCL)
- new net SDA: R?.1, U?.5 (SDA)
- new net ~{WC}: JP?.1 (A)
Other:
- note added: "2kb"
- note added: "I2C EEPROM"
- note added: "LED on WC?"
- note added: "QSPI Flash"
- note added: "Stores motion sequences or logged data."
- note added: "Stores system configuration parameters."
- title: QSPI Flash -> QSPI Flash & EEPROM
- moved on the sheet: C?, R?, U?

Commit message: Aux IO Changes
Parts:
- removed JP?: ~{EC}, Jumper:SolderJumper-2_P1.3mm_Bridged_RoundedPad1.0x1.5mm, symbol Jumper:SolderJumper_2_Bridged
- added D?: BLUE, Diode_SMD:D_0805_2012Metric, symbol Device:LED
- added R?: 220, Resistor_SMD:R_0603_1608Metric, symbol Device:R_US
Connections:
- net +3.3V: now also R?.1, R?.1
- net GND: no longer R?.2
- net ~{WC}: now also R?.2, U?.7 (~{WC}), D?.1 (K)
- new net: D?.2 (A), R?.2
Other:
- note removed: "LED on WC?"
- moved on the sheet: C?, JP?, R?, U?
